File: hardware/board/harp_treadmill.kicad_sch (KiCad schematic)
At the start: 0 parts

Commit message: update sch and pcb
Parts:
- added H1: MountingHole_Pad, kicad_component_library:Terminal_Keystone_779x_EdgeMount_Horizontal, symbol Mechanical:MountingHole_Pad
Connections:
- new net GND: H1.1
Other:
- note added: "Ground Lug"
- note removed: "FIXME: REF2033 bypass caps don't have footprints specified."
Changed lines of the file:
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@@
+    (stroke (width 0) (type default))
+  )
+  (wire (pts (xy 226.822 134.112) (xy 226.822 134.62))
     (stroke (width 0) (type default))
   )
@@
     (stroke (width 0) (type default))
   )
-  (text "FIXME: REF2033 bypass caps don't have footprints specified."
-    (at 118.11 141.605 0)
-    (effects (font (face "KiCad Font") (size 2 2) (thickness 0.4) bold) (justify left bottom))
-  )
   (text "TODO: consider 6V and 12V setting via resistors?\n    We could buffer the feedback resistor value into the\n    PICO's built-in ADC."
     (at 118.11 130.81 0)
     (effects (font (size 1.27 1.27)) (justify left bottom))
   )
+  (text "Ground Lug" (at 222.25 125.984 0)
+    (effects (font (size 1.27 1.27)) (justify left bottom))
+  )
+  (symbol (lib_id "Mechanical:MountingHole_Pad") (at 226.822 131.572 0) (unit 1)
+    (in_bom yes) (on_board yes) (dnp no) (fields_autoplaced)
+    (property "Reference" "H1" (at 229.87 130.302 0)
+      (effects (font (size 1.27 1.27)) (justify left))
+    )
+    (property "Value" "MountingHole_Pad" (at 229.87 131.572 0)
+      (effects (font (size 1.27 1.27)) (justify left) hide)
+    )
+    (property "Footprint" "kicad_component_library:Terminal_Keystone_779x_EdgeMount_Horizontal" (at 226.822 131.572 0)
+      (effects (font (size 1.27 1.27)) hide)
+    )
+    (property "Datasheet" "~" (at 226.822 131.572 0)
+      (effects (font (size 1.27 1.27)) hide)
+    )
+    (property "Link" "" (at 226.822 131.572 0)
+      (effects (font (size 1.27 1.27)) hide)
+    )
+    (pin "1")
+    (instances
+      (project "harp_treadmill"
+        (path "/e63e39d7-6ac0-4ffd-8aa3-1841a4541b55"
+          (reference "H1") (unit 1)
+        )
+      )
+    )
+  )
+  (symbol (lib_id "power:GND") (at 226.822 134.62 0) (unit 1)
+    (in_bom yes) (on_board yes) (dnp no) (fields_autoplaced)
+    (property "Reference" "#PWR0127" (at 226.822 140.97 0)
+      (effects (font (size 1.27 1.27)) hide)
+    )
+    (property "Value" "GND" (at 226.822 139.7 0)
+      (effects (font (size 1.27 1.27)))
+    )
+    (property "Footprint" "" (at 226.822 134.62 0)
+      (effects (font (size 1.27 1.27)) hide)
+    )
+    (property "Datasheet" "" (at 226.822 134.62 0)
+      (effects (font (size 1.27 1.27)) hide)
+    )
+    (pin "1")
+    (instances
+      (project "harp_treadmill"
+        (path "/e63e39d7-6ac0-4ffd-8aa3-1841a4541b55"
+          (reference "#PWR0127") (unit 1)
+        )
+      )
+    )
+  )
   (sheet (at 102.235 69.215) (size 15.875 20.32) (fields_autoplaced)
