File: hardware/board/torque_load_sensing.kicad_sch (KiCad schematic)
At the start: 21 parts

Commit message: update schematic
Parts:
- added C27: 100nF, Capacitor_SMD:C_0402_1005Metric, symbol Device:C
- D?: footprint (none) -> Diode_SMD:D_SOD-123F; Link (none) -> https://www.mouser.com/ProductDetail/Nexperia/BZT52H-A3V3-Q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; Manufacturer (none) -> Nexperia
Connections:
- net +3V3: now also C27.2
- net GND: now also C27.1
Other:
- note added: "ADS7049 Bypass Cap"
Changed lines of the file:
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@@
+    (stroke (width 0) (type default))
+  )
+  (wire (pts (xy 160.655 186.69) (xy 160.655 187.96))
     (stroke (width 0) (type default))
   )
@@
   )
   (wire (pts (xy 139.065 65.405) (xy 139.065 71.755))
+    (stroke (width 0) (type default))
+  )
+  (wire (pts (xy 160.655 177.8) (xy 160.655 179.07))
     (stroke (width 0) (type default))
   )
@@
   (text "See Signal Chain Basics #78 for more details on common mode voltage limitations.\nhttps://www.planetanalog.com/signal-chain-basics-78-how-to-avoid-common-mode-limitations-on-instrumentation-amplifiers/"
     (at 13.335 194.945 0)
+    (effects (font (size 1.27 1.27)) (justify left bottom))
+  )
+  (text "ADS7049\nBypass Cap" (at 156.21 170.18 0)
     (effects (font (size 1.27 1.27)) (justify left bottom))
   )
@@
     )
   )
+  (symbol (lib_id "power:GND") (at 160.655 187.96 0) (unit 1)
+    (in_bom yes) (on_board yes) (dnp no)
+    (property "Reference" "#PWR098" (at 160.655 194.31 0)
+      (effects (font (size 1.27 1.27)) hide)
+    )
+    (property "Value" "GND" (at 160.655 191.77 0)
+      (effects (font (size 1.27 1.27)))
+    )
+    (property "Footprint" "" (at 160.655 187.96 0)
+      (effects (font (size 1.27 1.27)) hide)
+    )
+    (property "Datasheet" "" (at 160.655 187.96 0)
+      (effects (font (size 1.27 1.27)) hide)
+    )
+    (pin "1")
+    (instances
+      (project "harp_treadmill"
+        (path "/e63e39d7-6ac0-4ffd-8aa3-1841a4541b55/45528c19-905b-4605-ba1b-282fdcb272c9"
+          (reference "#PWR098") (unit 1)
+        )
+        (path "/e63e39d7-6ac0-4ffd-8aa3-1841a4541b55/4d27c546-69b8-415d-ad57-797194b34e8d"
+          (reference "#PWR0105") (unit 1)
+        )
+        (path "/e63e39d7-6ac0-4ffd-8aa3-1841a4541b55/93b3207b-e1ce-46d7-a52b-3e8fb1ae6901"
+          (reference "#PWR0109") (unit 1)
+        )
+      )
+    )
+  )
   (symbol (lib_id "Connector:Conn_01x05_Female") (at 67.31 89.535 0) (mirror y) (unit 1)
     (in_bom yes) (on_board yes) (dnp no)
@@
       (effects (font (size 1.27 1.27)) (justify left))
     )
-    (property "Footprint" "" (at 165.735 94.615 0)
+    (property "Footprint" "Diode_SMD:D_SOD-123F" (at 165.735 94.615 0)
       (effects (font (size 1.27 1.27)) hide)
     )
@@
       (effects (font (size 1.27 1.27)) hide)
     )
+    (property "Link" "https://www.mouser.com/ProductDetail/Nexperia/BZT52H-A3V3-QX?qs=A6eO%252BMLsxmSzLn%252BZoY0yAg%3D%3D" (at 165.735 94.615 90)
+      (effects (font (size 1.27 1.27)) hide)
+    )
+    (property "Manufacturer" "Nexperia" (at 165.735 94.615 90)
+      (effects (font (size 1.27 1.27)) hide)
+    )
     (pin "1")
     (pin "2")
@@
         (path "/e63e39d7-6ac0-4ffd-8aa3-1841a4541b55/93b3207b-e1ce-46d7-a52b-3e8fb1ae6901"
           (reference "D?") (unit 1)
+        )
+      )
+    )
+  )
+  (symbol (lib_id "power:+3V3") (at 160.655 177.8 0) (mirror y) (unit 1)
+    (in_bom yes) (on_board yes) (dnp no)
+    (property "Reference" "#PWR?" (at 160.655 181.61 0)
+      (effects (font (size 1.27 1.27)) hide)
+    )
+    (property "Value" "+3V3" (at 163.195 173.99 0)
+      (effects (font (size 1.27 1.27)) (justify left))
+    )
+    (property "Footprint" "" (at 160.655 177.8 0)
+      (effects (font (size 1.27 1.27)) hide)
+    )
+    (property "Datasheet" "" (at 160.655 177.8 0)
+      (effects (font (size 1.27 1.27)) hide)
+    )
+    (pin "1")
+    (instances
+      (project "harp_treadmill"
+        (path "/e63e39d7-6ac0-4ffd-8aa3-1841a4541b55"
+          (reference "#PWR?") (unit 1)
+        )
+        (path "/e63e39d7-6ac0-4ffd-8aa3-1841a4541b55/93b3207b-e1ce-46d7-a52b-3e8fb1ae6901"
+          (reference "#PWR0108") (unit 1)
+        )
+        (path "/e63e39d7-6ac0-4ffd-8aa3-1841a4541b55/4d27c546-69b8-415d-ad57-797194b34e8d"
+          (reference "#PWR0106") (unit 1)
         )
       )
@@
         )
       )
+    )
+  )
+  (symbol (lib_id "Device:C") (at 160.655 182.88 180) (unit 1)
+    (in_bom yes) (on_board yes) (dnp no)
+    (property "Reference" "C27" (at 164.465 180.34 0)
+      (effects (font (size 1.27 1.27)) (justify left))
+    )
+    (property "Value" "100nF" (at 167.005 185.42 0)
+      (effects (font (size 1.27 1.27)) (justify left))
+    )
+    (property "Footprint" "Capacitor_SMD:C_0402_1005Metric" (at 159.6898 179.07 0)
+      (effects (font (size 1.27 1.27)) hide)
+    )
+    (property "Datasheet" "http://www.passivecomponent.com/wp-content/uploads/datasheet/WTC_MLCC_General_Purpose.pdf" (at 160.655 182.88 0)
+      (effects (font (size 1.27 1.27)) hide)
+    )
+    (property "Link" "https://www.digikey.com/en/products/detail/walsin-technology-corporation/0402B104K160CT/6707534" (at 160.655 182.88 0)
+      (effects (font (size 1.27 1.27)) hide)
+    )
+    (property "Manufacturer" "Walson Technology Corporation" (at 160.655 182.88 0)
+      (effects (font (size 1.27 1.27)) hide)
+    )
+    (property "Manufacturer Number" "0402B104K160CT" (at 160.655 182.88 0)
+      (effects (font (size 1.27 1.27)) hide)
+    )
+    (property "Rated Voltage" "16V" (at 160.655 182.88 0)
+      (effects (font (size 1.27 1.27)) hide)
+    )
+    (property "Temperature Coefficient" "X7R" (at 160.655 182.88 0)
+      (effects (font (size 1.27 1.27)) hide)
+    )
+    (property "Tolerance" "10%" (at 160.655 182.88 0)
+      (effects (font (size 1.27 1.27)) hide)
+    )
+    (property "PCBWay Link" "https://www.pcbway.com/components/detail/0402B104K160CT/307171/" (at 160.655 182.88 0)
+      (effects (font (size 1.27 1.27)) hide)
+    )
+    (pin "1")
+    (pin "2")
+    (instances
+      (project "harp_treadmill"
+        (path "/e63e39d7-6ac0-4ffd-8aa3-1841a4541b55/45528c19-905b-4605-ba1b-282fdcb272c9"
+          (reference "C27") (unit 1)
+        )
+        (path "/e63e39d7-6ac0-4ffd-8aa3-1841a4541b55/4d27c546-69b8-415d-ad57-797194b34e8d"
+          (reference "C31") (unit 1)
+        )
+        (path "/e63e39d7-6ac0-4ffd-8aa3-1841a4541b55/93b3207b-e1ce-46d7-a52b-3e8fb1ae6901"
+          (reference "C32") (unit 1)
+        )
+      )

Commit message: update pcb
Parts:
- U7: renamed from U?; symbol machine_agency_components:AD8221 -> kicad_component_library:AD8226
- gave numbers to parts that had none: 19
Connections:
- net GNDA is gone; now on net GND: C23.2, C24.1, C25.2, C26.1, D5.2 (A)

Commit message: update sch and pcb
Parts:
- C24, C26: Alternate (none) -> GRM21BR61H106KE43L; Link https://www.digikey.com/en/products/detail/kemet/T529P106M0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 -> https://www.digikey.com/en/products/detail/murata-electroni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; Manufacturer Kemet -> Murata Electronics; Manufacturer Number T529P106M010AAE200 -> GRM21BR61H106KE43L; Rated Voltage (none) -> 50V; Temperature Coefficient (none) -> X5R; Tolerance (none) -> 10%
- J3: footprint (none) -> Connector_Phoenix_MC:PhoenixContact_MC_1,5_5-G-3.5_1x05_P3.50mm_Horizontal; Alternate (none) -> 1844249; Link (none) -> https://www.mouser.com/ProductDetail/Phoenix-Contact/187629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; Manufacturer (none) -> Phoenix Contact; Manufacturer Number (none) -> 1876291
- R14, R8: footprint (none) -> Resistor_SMD:R_0402_1005Metric
Other:
- note added: "31.25[MHz] SPI"
- note added: "Use Phoenix Contact 3.5mm Plug pn 1840395"
- note removed: "Use Phoenix Contact 3.5mm Plug pn 1803578"
Changed lines of the file:
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@@
+    (effects (font (size 1.27 1.27)) (justify left bottom))
+  )
+  (text "31.25[MHz] SPI" (at 237.236 77.216 0)
     (effects (font (size 1.27 1.27)) (justify left bottom))
   )
@@
     (effects (font (size 1.27 1.27)) (justify left bottom))
   )
-  (text "Use Phoenix Contact 3.5mm Plug\npn 1803578" (at 30.48 105.41 0)
+  (text "Use Phoenix Contact 3.5mm Plug\npn 1840395" (at 30.48 105.41 0)
     (effects (font (size 1.27 1.27)) (justify left bottom))
   )
@@
       (effects (font (size 1.27 1.27)) hide)
     )
-    (property "Datasheet" "https://connect.kemet.com:7667/gateway/IntelliData-ComponentDocumentation/1.0/download/specsheet/T529P106M010AAE200" (at 144.145 112.395 0)
-      (effects (font (size 1.27 1.27)) hide)
-    )
-    (property "Link" "https://www.digikey.com/en/products/detail/kemet/T529P106M010AAE200/8582783" (at 144.145 112.395 90)
-      (effects (font (size 1.27 1.27)) hide)
-    )
-    (property "Manufacturer" "Kemet" (at 144.145 112.395 90)
-      (effects (font (size 1.27 1.27)) hide)
-    )
-    (property "Manufacturer Number" "T529P106M010AAE200" (at 144.145 112.395 90)
+    (property "Datasheet" "https://search.murata.co.jp/Ceramy/image/img/A01X/G101/ENG/GRM21BR61H106KE43-01A.pdf" (at 144.145 112.395 0)
+      (effects (font (size 1.27 1.27)) hide)
+    )
+    (property "Link" "https://www.digikey.com/en/products/detail/murata-electronics/GRM21BR61H106KE43L/10326316" (at 144.145 112.395 90)
+      (effects (font (size 1.27 1.27)) hide)
+    )
+    (property "Manufacturer" "Murata Electronics" (at 144.145 112.395 90)
+      (effects (font (size 1.27 1.27)) hide)
+    )
+    (property "Manufacturer Number" "GRM21BR61H106KE43L" (at 144.145 112.395 90)
+      (effects (font (size 1.27 1.27)) hide)
+    )
+    (property "Alternate" "GRM21BR61H106KE43L" (at 144.145 112.395 0)
+      (effects (font (size 1.27 1.27)) hide)
+    )
+    (property "Rated Voltage" "50V" (at 144.145 112.395 0)
+      (effects (font (size 1.27 1.27)) hide)
+    )
+    (property "Temperature Coefficient" "X5R" (at 144.145 112.395 0)
+      (effects (font (size 1.27 1.27)) hide)
+    )
+    (property "Tolerance" "10%" (at 144.145 112.395 0)
       (effects (font (size 1.27 1.27)) hide)
     )
@@
       (effects (font (size 1.27 1.27)) hide)
     )
-    (property "Footprint" "" (at 67.31 89.535 0)
-      (effects (font (size 1.27 1.27)) hide)
-    )
-    (property "Datasheet" "~" (at 67.31 89.535 0)
+    (property "Footprint" "Connector_Phoenix_MC:PhoenixContact_MC_1,5_5-G-3.5_1x05_P3.50mm_Horizontal" (at 67.31 89.535 0)
+      (effects (font (size 1.27 1.27)) hide)
+    )
+    (property "Datasheet" "n/a" (at 67.31 89.535 0)
+      (effects (font (size 1.27 1.27)) hide)
+    )
+    (property "Link" "https://www.mouser.com/ProductDetail/Phoenix-Contact/1876291?qs=z6e26OirEkwpKa%252BIKFEHGw%3D%3D" (at 67.31 89.535 0)
+      (effects (font (size 1.27 1.27)) hide)
+    )
+    (property "Manufacturer Number" "1876291" (at 67.31 89.535 0)
+      (effects (font (size 1.27 1.27)) hide)
+    )
+    (property "Manufacturer" "Phoenix Contact" (at 67.31 89.535 0)
+      (effects (font (size 1.27 1.27)) hide)
+    )
+    (property "Alternate" "1844249" (at 67.31 89.535 0)
       (effects (font (size 1.27 1.27)) hide)
     )
@@
       (effects (font (size 1.27 1.27)) hide)
     )
-    (property "Datasheet" "https://connect.kemet.com:7667/gateway/IntelliData-ComponentDocumentation/1.0/download/specsheet/T529P106M010AAE200" (at 144.145 71.755 0)
-      (effects (font (size 1.27 1.27)) hide)
-    )
-    (property "Link" "https://www.digikey.com/en/products/detail/kemet/T529P106M010AAE200/8582783" (at 144.145 71.755 90)
-      (effects (font (size 1.27 1.27)) hide)
-    )
-    (property "Manufacturer" "Kemet" (at 144.145 71.755 90)
-      (effects (font (size 1.27 1.27)) hide)
-    )
-    (property "Manufacturer Number" "T529P106M010AAE200" (at 144.145 71.755 90)
+    (property "Datasheet" "https://search.murata.co.jp/Ceramy/image/img/A01X/G101/ENG/GRM21BR61H106KE43-01A.pdf" (at 144.145 71.755 0)
+      (effects (font (size 1.27 1.27)) hide)
+    )
+    (property "Link" "https://www.digikey.com/en/products/detail/murata-electronics/GRM21BR61H106KE43L/10326316" (at 144.145 71.755 90)
+      (effects (font (size 1.27 1.27)) hide)
+    )
+    (property "Manufacturer" "Murata Electronics" (at 144.145 71.755 90)
+      (effects (font (size 1.27 1.27)) hide)
+    )
+    (property "Manufacturer Number" "GRM21BR61H106KE43L" (at 144.145 71.755 90)
+      (effects (font (size 1.27 1.27)) hide)
+    )
+    (property "Alternate" "GRM21BR61H106KE43L" (at 144.145 71.755 0)
+      (effects (font (size 1.27 1.27)) hide)
+    )
+    (property "Rated Voltage" "50V" (at 144.145 71.755 0)
+      (effects (font (size 1.27 1.27)) hide)
+    )
+    (property "Temperature Coefficient" "X5R" (at 144.145 71.755 0)
+      (effects (font (size 1.27 1.27)) hide)
+    )
+    (property "Tolerance" "10%" (at 144.145 71.755 0)
       (effects (font (size 1.27 1.27)) hide)
     )
@@
       (effects (font (size 1.27 1.27)))
     )
-    (property "Footprint" "" (at 98.425 91.567 90)
+    (property "Footprint" "Resistor_SMD:R_0402_1005Metric" (at 98.425 91.567 90)
       (effects (font (size 1.27 1.27)) hide)
     )
@@
       (effects (font (size 1.27 1.27)))
     )
-    (property "Footprint" "" (at 98.425 84.963 90)
-      (effects (font (size 1.27 1.27)) hide)
-    )
+    (property "Footprint" "Resistor_SMD:R_0402_1005Metric" (at 98.425 84.963 90)
+      (effects (font (size 1.27 1.27)) hide)
+    )

Commit message: update schematic; continue pcb draft
Parts:
- removed C23, C25: 0.1uF, symbol Device:C
- removed D5: D_Zener, Diode_SMD:D_SOD-123F, symbol Device:D_Zener
- removed R14, R8: 10K, Resistor_SMD:R_0402_1005Metric, symbol Device:R
- added C27, C58 (x2): 100nF, Capacitor_SMD:C_0402_1005Metric, symbol Device:C
- added R9: 10K, Resistor_SMD:R_0402_1005Metric, symbol Device:R
- added RN1: 20K, Resistor_SMD:R_Array_Convex_2x0606, symbol Device:R_Pack02_Split
- added U10: AD8615, Package_TO_SOT_SMD:TSOT-23-5, symbol kicad_component_library:AD8615
- C20, C22: footprint (none) -> Capacitor_SMD:C_0402_1005Metric; Link https://www.digikey.com/en/products/detail/murata-electroni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 -> https://www.digikey.com/en/products/detail/kyocera-avx/KGM0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; Manufacturer Murata Electronics -> KYOCERA AVX; Manufacturer Number GCM1555C1H101FA16D -> KGM05ACG1H101FH
- C21: footprint (none) -> Capacitor_SMD:C_0402_1005Metric; Link https://www.digikey.com/en/products/detail/murata-electronics/GCM1555C1H101FA16D/6605978 -> https://www.digikey.com/en/products/detail/murata-electronics/GRM1555C1H102JA01D/702509; Manufacturer Number GCM1555C1H101FA16D -> GRM1555C1H102JA01D
- C24, C26: Alternate GRM21BR61H106KE43L -> (none); Link https://www.digikey.com/en/products/detail/murata-electroni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 -> https://www.digikey.com/en/products/detail/kemet/T529P106M0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; Manufacturer Murata Electronics -> Kemet; Manufacturer Number GRM21BR61H106KE43L -> T529P106M010AAE200; Notes (none) -> polarized, anode band; Rated Voltage 50V -> 10V; Temperature Coefficient X5R -> (none); Tolerance 10% -> 20%
- R15: footprint Resistor_SMD:R_0603_1608Metric -> Resistor_SMD:R_0603_1608Metric_Pad0.98x0.95mm_HandSolder
Connections:
- net +3V3: now also C27.2, U10.5 (V+)
- net +5V: now also C24.1, C58.2; no longer C24.2
- net -5V: now also C58.2
- net GND: now also C24.2, C27.1, C58.1, C58.1, U10.2 (V-); no longer C24.1
- net at C20.2, C21.1, U7.1 (IN-): now also RN1.4 (R1.2)
- net at C21.2, C22.1, U7.4 (IN+): now also RN1.3 (R2.2)
- net at R16.2, TP1.1: now also U10.1, U10.4 (-); no longer U7.7 (VOUT)
- net at J3.2 (Pin_2): now also RN1.1 (R1.1)
- net at J3.3 (Pin_3): now also RN1.2 (R2.1)
- new net: R9.2, U7.7 (VOUT)
- new net: R9.1, U10.3 (+)
Other:
- note added: "AD8615 * clamps maximum output voltage. * sources sufficient current to ADC across full scale range."
- note added: "AD8615 Bypass Cap"
- note added: "F_{c com} = 1/(2πRC_{C}) = 7.957[KHz]"
- note added: "F_{c diff} = 1/(2πR(2C_{D} + C_{C})) = 6.631[KHz]"
- note added: "i_{out,max} = 13[mA]"
- note added: "i_{out,max} = 150[mA]"
- note removed: "3.3V 1% Clipper"
- note removed: "AD8226 has indefinite short-circuit current output of 13mA."
- note removed: "F_{c com} = 1/(2πRC_{C}) = 159.155KHz"
- note removed: "F_{c diff} = 1/(2πR(2C_{D} + C_{C})) = 7.579KHz"
- note removed: "Output Range: 0-3.3[V]"
- note removed: "See Signal Chain Basics #78 for more details on common mode voltage limitations. https://www.planetanalog.com/signal-chain-basics-78-how-to-avoid-common-mode-limitations-on-instrumentation-amplifiers/"
- note removed: "Tantalum"
- moved on the sheet: C26
