File: hardware/board/torque_load_driving.kicad_sch (KiCad schematic)
At the start: 21 parts, among them U1 ADS7049

Commit message: update pcb
Parts:
- removed C?: 0.1uF, symbol Device:C
- added C27: 100nF, Capacitor_SMD:C_0402_1005Metric, symbol Device:C
- U11: renamed from U?; symbol machine_agency_components:INA180 -> kicad_component_library:INA180
- U12: renamed from U?; symbol machine_agency_components:UCC27537 -> kicad_component_library:UCC27537
- gave numbers to parts that had none: 6
Connections:
- net +3V3: now also C27.2
- net GND: now also C27.1
Changed lines of the file:
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@@
   (symbol (lib_id "Device:D") (at 189.865 101.6 270) (unit 1)
     (in_bom yes) (on_board yes) (dnp no)
-    (property "Reference" "D?" (at 185.42 99.06 90)
+    (property "Reference" "D6" (at 185.42 99.06 90)
       (effects (font (size 1.27 1.27)) (justify left))
     )
@@
       (project "harp_treadmill"
         (path "/e63e39d7-6ac0-4ffd-8aa3-1841a4541b55/4d27c546-69b8-415d-ad57-797194b34e8d"
-          (reference "D?") (unit 1)
+          (reference "D6") (unit 1)
         )
       )
@@
         )
         (path "/e63e39d7-6ac0-4ffd-8aa3-1841a4541b55/4d27c546-69b8-415d-ad57-797194b34e8d"
-          (reference "R?") (unit 1)
+          (reference "R24") (unit 1)
         )
       )
@@
   (symbol (lib_id "kicad_component_library:AD8615") (at 134.62 86.36 0) (mirror y) (unit 1)
     (in_bom yes) (on_board yes) (dnp no)
-    (property "Reference" "U?" (at 131.445 82.55 0)
+    (property "Reference" "U10" (at 131.445 82.55 0)
       (effects (font (size 1.27 1.27)) (justify right))
     )
@@
       (project "harp_treadmill"
         (path "/e63e39d7-6ac0-4ffd-8aa3-1841a4541b55/4d27c546-69b8-415d-ad57-797194b34e8d"
-          (reference "U?") (unit 1)
+          (reference "U10") (unit 1)
         )
       )
@@
   (symbol (lib_id "Connector:Conn_01x02_Female") (at 197.485 100.33 0) (unit 1)
     (in_bom yes) (on_board yes) (dnp no)
-    (property "Reference" "J?" (at 196.85 98.425 0)
+    (property "Reference" "J4" (at 196.85 98.425 0)
       (effects (font (size 1.27 1.27)) (justify left))
     )
@@
       (project "harp_treadmill"
         (path "/e63e39d7-6ac0-4ffd-8aa3-1841a4541b55/4d27c546-69b8-415d-ad57-797194b34e8d"
-          (reference "J?") (unit 1)
+          (reference "J4") (unit 1)
         )
       )
@@
     )
   )
+  (symbol (lib_id "Device:C") (at 20.32 181.61 180) (unit 1)
+    (in_bom yes) (on_board yes) (dnp no)
+    (property "Reference" "C27" (at 24.13 179.07 0)
+      (effects (font (size 1.27 1.27)) (justify left))
+    )
+    (property "Value" "100nF" (at 26.67 184.15 0)
+      (effects (font (size 1.27 1.27)) (justify left))
+    )
+    (property "Footprint" "Capacitor_SMD:C_0402_1005Metric" (at 19.3548 177.8 0)
+      (effects (font (size 1.27 1.27)) hide)
+    )
+    (property "Datasheet" "http://www.passivecomponent.com/wp-content/uploads/datasheet/WTC_MLCC_General_Purpose.pdf" (at 20.32 181.61 0)
+      (effects (font (size 1.27 1.27)) hide)
+    )
+    (property "Link" "https://www.digikey.com/en/products/detail/walsin-technology-corporation/0402B104K160CT/6707534" (at 20.32 181.61 0)
+      (effects (font (size 1.27 1.27)) hide)
+    )
+    (property "Manufacturer" "Walson Technology Corporation" (at 20.32 181.61 0)
+      (effects (font (size 1.27 1.27)) hide)
+    )
+    (property "Manufacturer Number" "0402B104K160CT" (at 20.32 181.61 0)
+      (effects (font (size 1.27 1.27)) hide)
+    )
+    (property "Rated Voltage" "16V" (at 20.32 181.61 0)
+      (effects (font (size 1.27 1.27)) hide)
+    )
+    (property "Temperature Coefficient" "X7R" (at 20.32 181.61 0)
+      (effects (font (size 1.27 1.27)) hide)
+    )
+    (property "Tolerance" "10%" (at 20.32 181.61 0)
+      (effects (font (size 1.27 1.27)) hide)
+    )
+    (property "PCBWay Link" "https://www.pcbway.com/components/detail/0402B104K160CT/307171/" (at 20.32 181.61 0)
+      (effects (font (size 1.27 1.27)) hide)
+    )
+    (pin "1")
+    (pin "2")
+    (instances
+      (project "harp_treadmill"
+        (path "/e63e39d7-6ac0-4ffd-8aa3-1841a4541b55/45528c19-905b-4605-ba1b-282fdcb272c9"
+          (reference "C27") (unit 1)
+        )
+        (path "/e63e39d7-6ac0-4ffd-8aa3-1841a4541b55/4d27c546-69b8-415d-ad57-797194b34e8d"
+          (reference "C59") (unit 1)
+        )
+      )
+    )
+  )
   (symbol (lib_id "power:GND") (at 161.925 135.89 0) (mirror y) (unit 1)
     (in_bom yes) (on_board yes) (dnp no)
@@
         )
         (path "/e63e39d7-6ac0-4ffd-8aa3-1841a4541b55/4d27c546-69b8-415d-ad57-797194b34e8d"
-          (reference "R?") (unit 1)
+          (reference "R23") (unit 1)
         )
       )
@@
         )
         (path "/e63e39d7-6ac0-4ffd-8aa3-1841a4541b55/4d27c546-69b8-415d-ad57-797194b34e8d"
-          (reference "R?") (unit 1)
+          (reference "R25") (unit 1)
         )
       )
@@
         )
         (path "/e63e39d7-6ac0-4ffd-8aa3-1841a4541b55/4d27c546-69b8-415d-ad57-797194b34e8d"
-          (reference "U?") (unit 1)
-        )
-      )
-    )
-  )
-  (symbol (lib_id "machine_agency_components:UCC27537") (at 161.925 124.46 0) (unit 1)
-    (in_bom yes) (on_board yes) (dnp no)
-    (property "Reference" "U?" (at 156.845 115.57 0)
+          (reference "U9") (unit 1)
+        )
+      )
+    )
+  )
+  (symbol (lib_id "kicad_component_library:UCC27537") (at 161.925 124.46 0) (unit 1)
+    (in_bom yes) (on_board yes) (dnp no)
+    (property "Reference" "U12" (at 156.845 115.57 0)
       (effects (font (size 1.27 1.27)))
     )
@@
       (project "harp_treadmill"
         (path "/e63e39d7-6ac0-4ffd-8aa3-1841a4541b55/4d27c546-69b8-415d-ad57-797194b34e8d"
-          (reference "U?") (unit 1)
+          (reference "U12") (unit 1)
         )
       )
@@
   (symbol (lib_id "Transistor_FET:IRF7403") (at 187.325 124.46 0) (unit 1)
     (in_bom yes) (on_board yes) (dnp no)
-    (property "Reference" "Q?" (at 191.135 121.285 0)
+    (property "Reference" "Q1" (at 191.135 121.285 0)
       (effects (font (size 1.27 1.27)) (justify left))
     )
@@
       (project "harp_treadmill"
         (path "/e63e39d7-6ac0-4ffd-8aa3-1841a4541b55/4d27c546-69b8-415d-ad57-797194b34e8d"
-          (reference "Q?") (unit 1)
+          (reference "Q1") (unit 1)
         )
       )
@@
         )
         (path "/e63e39d7-6ac0-4ffd-8aa3-1841a4541b55/4d27c546-69b8-415d-ad57-797194b34e8d"
-          (reference "R?") (unit 1)
-        )
-      )
-    )
-  )
-  (symbol (lib_id "Device:C") (at 20.32 181.61 0) (unit 1)
-    (in_bom yes) (on_board yes) (dnp no) (fields_autoplaced)
-    (property "Reference" "C?" (at 24.13 180.3399 0)
-      (effects (font (size 1.27 1.27)) (justify left))
-    )
-    (property "Value" "0.1uF" (at 24.13 182.8799 0)
-      (effects (font (size 1.27 1.27)) (justify left))
-    )
-    (property "Footprint" "" (at 21.2852 185.42 0)
-      (effects (font (size 1.27 1.27)) hide)
-    )
-    (property "Datasheet" "~" (at 20.32 181.61 0)
-      (effects (font (size 1.27 1.27)) hide)
-    )
-    (pin "1")
-    (pin "2")
-    (instances
-      (project "harp_treadmill"
-        (path "/e63e39d7-6ac0-4ffd-8aa3-1841a4541b55"
-          (reference "C?") (unit 1)
-        )
-        (path "/e63e39d7-6ac0-4ffd-8aa3-1841a4541b55/4d27c546-69b8-415d-ad57-797194b34e8d"
-          (reference "C1") (unit 1)
+          (reference "R21") (unit 1)
         )
       )
@@
     )
   )
-  (symbol (lib_id "machine_agency_components:INA180") (at 161.925 86.36 0) (mirror y) (unit 1)
-    (in_bom yes) (on_board yes) (dnp no)
-    (property "Reference" "U?" (at 157.48 82.55 0)
+  (symbol (lib_id "kicad_component_library:INA180") (at 161.925 86.36 0) (mirror y) (unit 1)
+    (in_bom yes) (on_board yes) (dnp no)
+    (property "Reference" "U11" (at 157.48 82.55 0)
       (effects (font (size 1.27 1.27)))
     )
@@
       (project "harp_treadmill"
         (path "/e63e39d7-6ac0-4ffd-8aa3-1841a4541b55/4d27c546-69b8-415d-ad57-797194b34e8d"
-          (reference "U?") (unit 1)
+          (reference "U11") (unit 1)
         )
       )
@@
   (symbol (lib_id "Device:R") (at 189.865 86.36 0) (mirror y) (unit 1)
     (in_bom yes) (on_board yes) (dnp no)
-    (property "Reference" "R?" (at 192.405 85.0899 0)
+    (property "Reference" "R27" (at 192.405 85.0899 0)
       (effects (font (size 1.27 1.27)) (justify right))
     )
@@
       (project "harp_treadmill"
         (path "/e63e39d7-6ac0-4ffd-8aa3-1841a4541b55/4d27c546-69b8-415d-ad57-797194b34e8d"
-          (reference "R?") (unit 1)
+          (reference "R27") (unit 1)
         )
       )
@@
   (symbol (lib_id "Device:R") (at 177.165 124.46 90) (unit 1)
     (in_bom yes) (on_board yes) (dnp no)
-    (property "Reference" "R?" (at 177.165 127 90)
+    (property "Reference" "R26" (at 177.165 127 90)
       (effects (font (size 1.27 1.27)))
     )
@@
       (project "harp_treadmill"
         (path "/e63e39d7-6ac0-4ffd-8aa3-1841a4541b55/4d27c546-69b8-415d-ad57-797194b34e8d"
-          (reference "R?") (unit 1)
+          (reference "R26") (unit 1)
         )
       )
@@
   (symbol (lib_id "power:+3V3") (at 161.925 77.47 0) (mirror y) (unit 1)
     (in_bom yes) (on_board yes) (dnp no)
-    (property "Reference" "#PWR?" (at 161.925 81.28 0)
+    (property "Reference" "#PWR0123" (at 161.925 81.28 0)
       (effects (font (size 1.27 1.27)) hide)
     )
@@
       (project "harp_treadmill"
         (path "/e63e39d7-6ac0-4ffd-8aa3-1841a4541b55/4d27c546-69b8-415d-ad57-797194b34e8d"
-          (reference "#PWR?") (unit 1)
+          (reference "#PWR0123") (unit 1)
         )
       )
@@
         )
         (path "/e63e39d7-6ac0-4ffd-8aa3-1841a4541b55/4d27c546-69b8-415d-ad57-797194b34e8d"
-          (reference "R?") (unit 1)
+          (reference "R22") (unit 1)
         )
       )
@@
         )
         (path "/e63e39d7-6ac0-4ffd-8aa3-1841a4541b55/4d27c546-69b8-415d-ad57-797194b34e8d"
-          (reference "C?") (unit 1)
-        )
-      )
+          (reference "C33") (unit 1)
+        )
+      )

Commit message: update sch and pcb
Parts:
- added C26: 10uF, Capacitor_SMD:C_0805_2012Metric, symbol Device:C
- C26: Alternate CL21B106KOQNNNE -> GRM21BR61H106KE43L; Link https://www.digikey.com/en/products/detail/murata-electronics/GRM21BZ71E106KE15L/13904911 -> https://www.digikey.com/en/products/detail/murata-electronics/GRM21BR61H106KE43L/10326316; Manufacturer Number GRM21BZ71E106KE15L -> GRM21BR61H106KE43L; Rated Voltage 25V -> 50V; Temperature Coefficient X7R -> X5R; Tolerance (none) -> 10%
- J4: footprint (none) -> Connector_Phoenix_MC:PhoenixContact_MC_1,5_2-G-3.5_1x02_P3.50mm_Horizontal; Link (none) -> https://www.digikey.com/en/products/detail/phoenix-contact/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; Manufacturer (none) -> Phoenix Contact; Manufacturer Number (none) -> 1844210
Connections:
- net +12V: now also C26.1
- net GND: now also C26.2
Other:
- note added: "31.25[MHz] SPI"
- note added: "Brake Bypass Cap"
- note added: "Floating BRAKE_PWM signal = Output LOW"
- note added: "Mates with: 1894655"
- note added: "Max PWM Frequency: 200[KHz]"
- note removed: "Floating IN signal = Output LOW"
- note removed: "Max PWM Frequency: 100[KHz]"
Changed lines of the file:
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@@
+    (stroke (width 0) (type default))
+  )
+  (wire (pts (xy 131.318 185.42) (xy 131.318 186.69))
     (stroke (width 0) (type default))
   )
@@
   )
   (wire (pts (xy 189.865 110.49) (xy 189.865 119.38))
+    (stroke (width 0) (type default))
+  )
+  (wire (pts (xy 131.318 176.53) (xy 131.318 177.8))
     (stroke (width 0) (type default))
   )
@@
     (effects (font (size 1.27 1.27)) (justify left bottom))
   )
+  (text "31.25[MHz] SPI" (at 59.436 78.994 0)
+    (effects (font (size 1.27 1.27)) (justify left bottom))
+  )
+  (text "Brake\nBypass Cap" (at 128.27 168.656 0)
+    (effects (font (size 1.27 1.27)) (justify left bottom))
+  )
   (text "U13 must be driven by a low impedance source \nand requires ~300pF input capacitance for stability."
     (at 101.6 111.76 0)
@@
     (effects (font (size 1.27 1.27)) (justify left bottom))
   )
-  (text "Floating IN signal = Output LOW" (at 120.015 129.54 0)
+  (text "Mates with: 1894655" (at 214.63 102.235 0)
     (effects (font (size 1.27 1.27)) (justify left bottom))
   )
-  (text "Max PWM Frequency: 100[KHz]" (at 120.015 132.08 0)
+  (text "Floating BRAKE_PWM signal = Output LOW" (at 108.712 129.794 0)
+    (effects (font (size 1.27 1.27)) (justify left bottom))
+  )
+  (text "Max PWM Frequency: 200[KHz]" (at 120.015 132.08 0)
     (effects (font (size 1.27 1.27)) (justify left bottom))
   )
@@
       (effects (font (size 1.27 1.27)) hide)
     )
-    (property "Datasheet" "https://search.murata.co.jp/Ceramy/image/img/A01X/G101/ENG/GRM21BZ71E106KE15-01.pdf" (at 41.91 181.61 0)
-      (effects (font (size 1.27 1.27)) hide)
-    )
-    (property "Link" "https://www.digikey.com/en/products/detail/murata-electronics/GRM21BZ71E106KE15L/13904911" (at 41.91 181.61 0)
-      (effects (font (size 1.27 1.27)) hide)
-    )
-    (property "Manufacturer Number" "GRM21BZ71E106KE15L" (at 41.91 181.61 0)
-      (effects (font (size 1.27 1.27)) hide)
-    )
-    (property "Rated Voltage" "25V" (at 41.91 181.61 0)
-      (effects (font (size 1.27 1.27)) hide)
-    )
-    (property "Temperature Coefficient" "X7R" (at 41.91 181.61 0)
+    (property "Datasheet" "https://search.murata.co.jp/Ceramy/image/img/A01X/G101/ENG/GRM21BR61H106KE43-01A.pdf" (at 41.91 181.61 0)
+      (effects (font (size 1.27 1.27)) hide)
+    )
+    (property "Link" "https://www.digikey.com/en/products/detail/murata-electronics/GRM21BR61H106KE43L/10326316" (at 41.91 181.61 0)
+      (effects (font (size 1.27 1.27)) hide)
+    )
+    (property "Manufacturer Number" "GRM21BR61H106KE43L" (at 41.91 181.61 0)
+      (effects (font (size 1.27 1.27)) hide)
+    )
+    (property "Rated Voltage" "50V" (at 41.91 181.61 0)
+      (effects (font (size 1.27 1.27)) hide)
+    )
+    (property "Temperature Coefficient" "X5R" (at 41.91 181.61 0)
       (effects (font (size 1.27 1.27)) hide)
     )
@@
       (effects (font (size 1.27 1.27)) hide)
     )
-    (property "Alternate" "CL21B106KOQNNNE" (at 41.91 181.61 0)
+    (property "Alternate" "GRM21BR61H106KE43L" (at 41.91 181.61 0)
+      (effects (font (size 1.27 1.27)) hide)
+    )
+    (property "Tolerance" "10%" (at 41.91 181.61 0)
       (effects (font (size 1.27 1.27)) hide)
     )
@@
       (effects (font (size 1.27 1.27)) (justify left) hide)
     )
-    (property "Footprint" "" (at 197.485 100.33 0)
+    (property "Footprint" "Connector_Phoenix_MC:PhoenixContact_MC_1,5_2-G-3.5_1x02_P3.50mm_Horizontal" (at 197.485 100.33 0)
       (effects (font (size 1.27 1.27)) hide)
     )
     (property "Datasheet" "~" (at 197.485 100.33 0)
+      (effects (font (size 1.27 1.27)) hide)
+    )
+    (property "Manufacturer" "Phoenix Contact" (at 197.485 100.33 0)
+      (effects (font (size 1.27 1.27)) hide)
+    )
+    (property "Manufacturer Number" "1844210" (at 197.485 100.33 0)
+      (effects (font (size 1.27 1.27)) hide)
+    )
+    (property "Link" "https://www.digikey.com/en/products/detail/phoenix-contact/1844210/349195" (at 197.485 100.33 0)
       (effects (font (size 1.27 1.27)) hide)
     )
@@
         (path "/e63e39d7-6ac0-4ffd-8aa3-1841a4541b55/4d27c546-69b8-415d-ad57-797194b34e8d"
           (reference "#PWR0101") (unit 1)
+        )
+      )
+    )
+  )
+  (symbol (lib_id "power:GND") (at 131.318 186.69 0) (unit 1)
+    (in_bom yes) (on_board yes) (dnp no)
+    (property "Reference" "#PWR096" (at 131.318 193.04 0)
+      (effects (font (size 1.27 1.27)) hide)
+    )
+    (property "Value" "GND" (at 131.318 190.5 0)
+      (effects (font (size 1.27 1.27)))
+    )
+    (property "Footprint" "" (at 131.318 186.69 0)
+      (effects (font (size 1.27 1.27)) hide)
+    )
+    (property "Datasheet" "" (at 131.318 186.69 0)
+      (effects (font (size 1.27 1.27)) hide)
+    )
+    (pin "1")
+    (instances
+      (project "harp_treadmill"
+        (path "/e63e39d7-6ac0-4ffd-8aa3-1841a4541b55/45528c19-905b-4605-ba1b-282fdcb272c9"
+          (reference "#PWR096") (unit 1)
+        )
+        (path "/e63e39d7-6ac0-4ffd-8aa3-1841a4541b55/4d27c546-69b8-415d-ad57-797194b34e8d"
+          (reference "#PWR0129") (unit 1)
         )
       )
@@
     )
   )
+  (symbol (lib_id "power:+12V") (at 131.318 176.53 0) (unit 1)
+    (in_bom yes) (on_board yes) (dnp no) (fields_autoplaced)
+    (property "Reference" "#PWR015" (at 131.318 180.34 0)
+      (effects (font (size 1.27 1.27)) hide)
+    )
+    (property "Value" "+12V" (at 131.318 172.085 0)
+      (effects (font (size 1.27 1.27)))
+    )
+    (property "Footprint" "" (at 131.318 176.53 0)
+      (effects (font (size 1.27 1.27)) hide)
+    )
+    (property "Datasheet" "" (at 131.318 176.53 0)
+      (effects (font (size 1.27 1.27)) hide)
+    )
+    (pin "1")
+    (instances
+      (project "harp_treadmill"
+        (path "/e63e39d7-6ac0-4ffd-8aa3-1841a4541b55/1f049e4e-eb8d-47d9-901f-1dd446bfea55"
+          (reference "#PWR015") (unit 1)
+        )
+        (path "/e63e39d7-6ac0-4ffd-8aa3-1841a4541b55/4d27c546-69b8-415d-ad57-797194b34e8d"
+          (reference "#PWR0128") (unit 1)
+        )
+      )
+    )
+  )
   (symbol (lib_id "Device:C") (at 106.68 181.61 180) (unit 1)
     (in_bom yes) (on_board yes) (dnp no)
@@
         )
       )
+    )
+  )
+  (symbol (lib_id "Device:C") (at 131.318 181.61 0) (unit 1)
+    (in_bom yes) (on_board yes) (dnp no)
+    (property "Reference" "C26" (at 132.588 179.07 0)
+      (effects (font (size 1.27 1.27)) (justify left))
+    )
+    (property "Value" "10uF" (at 132.588 184.15 0)
+      (effects (font (size 1.27 1.27)) (justify left))
+    )
+    (property "Footprint" "Capacitor_SMD:C_0805_2012Metric" (at 132.2832 185.42 0)
+      (effects (font (size 1.27 1.27)) hide)
+    )
+    (property "Datasheet" "https://search.murata.co.jp/Ceramy/image/img/A01X/G101/ENG/GRM21BR61H106KE43-01A.pdf" (at 131.318 181.61 0)
+      (effects (font (size 1.27 1.27)) hide)
+    )
+    (property "Link" "https://www.digikey.com/en/products/detail/murata-electronics/GRM21BR61H106KE43L/10326316" (at 131.318 181.61 0)
+      (effects (font (size 1.27 1.27)) hide)
+    )
+    (property "Manufacturer Number" "GRM21BR61H106KE43L" (at 131.318 181.61 0)
+      (effects (font (size 1.27 1.27)) hide)
+    )
+    (property "Rated Voltage" "50V" (at 131.318 181.61 0)
+      (effects (font (size 1.27 1.27)) hide)
+    )
+    (property "Temperature Coefficient" "X5R" (at 131.318 181.61 0)
+      (effects (font (size 1.27 1.27)) hide)
+    )
+    (property "Manufacturer" "Murata Electronics" (at 131.318 181.61 0)
+      (effects (font (size 1.27 1.27)) hide)
+    )
+    (property "Alternate" "GRM21BR61H106KE43L" (at 131.318 181.61 0)
+      (effects (font (size 1.27 1.27)) hide)
+    )
+    (property "Tolerance" "10%" (at 131.318 181.61 0)
+      (effects (font (size 1.27 1.27)) hide)
+    )
+    (pin "1")
+    (pin "2")
+    (instances
+      (project "harp_treadmill"
+        (path "/e63e39d7-6ac0-4ffd-8aa3-1841a4541b55/45528c19-905b-4605-ba1b-282fdcb272c9"
+          (reference "C26") (unit 1)
+        )
+        (path "/e63e39d7-6ac0-4ffd-8aa3-1841a4541b55/4d27c546-69b8-415d-ad57-797194b34e8d"
+          (reference "C62") (unit 1)
+        )
+      )

Commit message: update schematic; continue pcb draft
Other:
- note added: "AD8615 sources sufficient current to ADC across full scale range."
Changed lines of the file:
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@@
     (effects (font (size 1.27 1.27)) (justify right bottom))
+  )
+  (text "AD8615 sources sufficient current \nto ADC across full scale range."
+    (at 126.365 106.68 0)
+    (effects (font (size 1.27 1.27)) (justify left bottom))
   )
   (text "Settling Time Summary:\n* INA180: 5[us]" (at 241.3 146.05 0)
