File: hardware/board/harp_core_rp2040_w_isolated_usb.kicad_sch (KiCad schematic)
At the start: 49 parts, among them J1 Conn_01x03_Male, J2 AudioJack3, J5 USB_C_Receptacle_USB2.0, U2 TPD2EUSB30, U3 ADUM4160, U4 RP2040, U5 W25Q16JVUXIQ, X1 ECS-TXO-2016

Commit message: update silkscreen size; add mating connector note
Parts:
- J2: footprint Connector_Audio:Jack_3.5mm_CUI_SJ-3523-SMT_Horizontal -> Connector_Audio:Jack_3.5mm_CUI_SJ-3524-SMT_Horizontal; Alternat (none) -> SJ-3523-SMT-TR; Link https://www.digikey.com/en/products/detail/cui-devices/SJ-3523-SMT-TR/281297 -> https://www.digikey.com/en/products/detail/cui-devices/SJ-3524-SMT-TR/281298; Manufacturer Number SJ-3523-SMT-TR -> SJ-3524-SMT-TR; PCBWay Link https://www.pcbway.com/components/detail/SJ3523SMTTR/473228/ -> (none)
- SW1: Notes washable -> aqueous washable
